File: schematics/oled-display-schematic.sch (KiCad schematic (older format))
At the start: 6 parts, among them J1 Left rail ESP32 devkit v1, J2 Right rail ESP32 devkit v1, J3 PCD8544 display, SW1 NO

Commit message: Fix resistor value
Parts:
- R1: value 5.6k -> 220k
Changed lines of the file:
@@
 P 4800 3100
 F 0 "R1" H 4730 3054 50  0000 R CNN
-F 1 "5.6k" H 4730 3145 50  0000 R CNN
+F 1 "220k" H 4730 3145 50  0000 R CNN
 F 2 "" V 4730 3100 50  0001 C CNN
 F 3 "~" H 4800 3100 50  0001 C CNN
